File: kitten6/kitten6.kicad_sch (KiCad schematic)
At the start: 10 parts, among them SW1 SW_Push, SW2 SW_Push, SW3 SW_Push, SW4 SW_Push, SW5 SW_Push, SW6 SW_Push, SW7 SW_Push, SW8 SW_Push, U1 Pico

Commit message: Change keypad layout
Parts:
- added SW9: SW_Push, MX_Hotswap:MX-Hotswap-1U, symbol Switch:SW_Push
- SW7: footprint MX_Hotswap:MX-Hotswap-2U -> MX_Hotswap:MX-Hotswap-1U
Connections:
- net GND: now also SW9.1
- net sw8: now reaches U1.11 (GPIO8)
- net sw8: now also SW9.2
Changed lines of the file:
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@@
+    (stroke (width 0) (type default) (color 0 0 0 0))
+  )
+  (wire (pts (xy 146.05 91.44) (xy 148.59 91.44))
     (stroke (width 0) (type default) (color 0 0 0 0))
   )
@@
     )
   )
+  (global_label "sw8" (shape input) (at 158.75 91.44 0) (fields_autoplaced)
+    (effects (font (size 1.27 1.27)) (justify left))
+    (property "Intersheet References" "${INTERSHEET_REFS}" (id 0) (at 164.7312 91.3606 0)
+      (effects (font (size 1.27 1.27)) (justify left) hide)
+    )
+  )
   (global_label "sw3" (shape input) (at 133.35 91.44 180) (fields_autoplaced)
     (effects (font (size 1.27 1.27)) (justify right))
@@
     (effects (font (size 1.27 1.27)) (justify right))
     (property "Intersheet References" "${INTERSHEET_REFS}" (id 0) (at 127.3688 104.0606 0)
+      (effects (font (size 1.27 1.27)) (justify right) hide)
+    )
+  )
+  (global_label "sw8" (shape input) (at 64.77 73.66 180) (fields_autoplaced)
+    (effects (font (size 1.27 1.27)) (justify right))
+    (property "Intersheet References" "${INTERSHEET_REFS}" (id 0) (at 58.7888 73.7394 0)
       (effects (font (size 1.27 1.27)) (justify right) hide)
     )
@@
     (property "Reference" "SW7" (id 0) (at 153.67 58.42 0))
     (property "Value" "SW_Push" (id 1) (at 153.67 60.96 0))
-    (property "Footprint" "MX_Hotswap:MX-Hotswap-2U" (id 2) (at 153.67 60.96 0)
+    (property "Footprint" "MX_Hotswap:MX-Hotswap-1U" (id 2) (at 153.67 60.96 0)
       (effects (font (size 1.27 1.27)) hide)
     )
@@
     (pin "2")
   )
+  (symbol (lib_id "Switch:SW_Push") (at 153.67 91.44 0) (unit 1)
+    (in_bom yes) (on_board yes) (fields_autoplaced)
+    (property "Reference" "SW9" (id 0) (at 153.67 83.82 0))
+    (property "Value" "SW_Push" (id 1) (at 153.67 86.36 0))
+    (property "Footprint" "MX_Hotswap:MX-Hotswap-1U" (id 2) (at 153.67 86.36 0)
+      (effects (font (size 1.27 1.27)) hide)
+    )
+    (property "Datasheet" "~" (id 3) (at 153.67 86.36 0)
+      (effects (font (size 1.27 1.27)) hide)
+    )
+    (pin "1")
+    (pin "2")
+  )
   (symbol (lib_id "power:GND") (at 82.55 114.3 0) (unit 1)
     (in_bom yes) (on_board yes) (fields_autoplaced)
@@
     )
     (path "/31098065-9db1-4578-b7a3-5a4f1cdc391c"
-      (reference "SW7") (unit 1) (value "SW_Push") (footprint "MX_Hotswap:MX-Hotswap-2U")
+      (reference "SW7") (unit 1) (value "SW_Push") (footprint "MX_Hotswap:MX-Hotswap-1U")
     )
     (path "/ab0512e1-4c7b-4ce7-a44e-5c66667242d9"
       (reference "SW8") (unit 1) (value "SW_Push") (footprint "MX_Hotswap:MX-Hotswap-1U")
     )
+    (path "/ef515edd-ce7f-4439-a4a0-ab64091c7c39"
+      (reference "SW9") (unit 1) (value "SW_Push") (footprint "MX_Hotswap:MX-Hotswap-1U")
+    )
     (path "/c990c3bb-baee-41f4-b8a6-4ab12f343b22"
