File: kneadpad9/kneadpad9.kicad_sch (KiCad schematic)
At the start: 11 parts, among them SW1 SW_Push, SW2 SW_Push, SW3 SW_Push, SW4 SW_Push, SW5 SW_Push, SW6 SW_Push, SW7 SW_Push, SW8 SW_Push, SW9 SW_Push, U1 Pico

Commit message: Add M2 mounting holes for backplate
Other:
- title: (none) -> KneadPad9
Changed lines of the file:
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@@
 (kicad_sch (version 20211123) (generator eeschema)
   (paper "A4")
+  (title_block
+    (title "KneadPad9")
+    (rev "1")
+  )
   (junction (at 146.05 66.04) (diameter 0) (color 0 0 0 0)
   )
