File: kneadpad9/kneadpad9.kicad_pcb (KiCad board)
At the start: 2 copper layers, 81.8 x 57.2 mm, 15 parts, among them SW1 SW_Push, SW2 SW_Push, SW3 SW_Push, SW4 SW_Push, SW5 SW_Push, SW6 SW_Push, SW7 SW_Push, SW8 SW_Push, SW9 SW_Push, U1 Pico

Commit message: Add placeholder label for JLC order
Other:
- board text added: "JLCJLCJLCJLC"
Changed lines of the file:
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@@
       (layerselection 0x00010fc_ffffffff)
       (disableapertmacros false)
-      (usegerberextensions false)
+      (usegerberextensions true)
       (usegerberattributes true)
       (usegerberadvancedattributes true)
-      (creategerberjobfile true)
+      (creategerberjobfile false)
       (svguseinch false)
       (svgprecision 6)
@@
       (psa4output false)
       (plotreference true)
-      (plotvalue true)
+      (plotvalue false)
       (plotinvisibletext false)
       (sketchpadsonfab false)
@@
   (gr_arc (start 100.24375 62) (mid 100.829536 60.585786) (end 102.24375 60) (layer "Edge.Cuts") (width 0.1))
   (gr_line (start 102.24375 117.15) (end 180 117.15) (layer "Edge.Cuts") (width 0.1))
+  (gr_text "JLCJLCJLCJLC" (at 101 61.5) (layer "B.SilkS")
+    (effects (font (size 1 1) (thickness 0.15)) (justify right mirror))
+  )
   (gr_text "KneadPad9 Rev.1 PCB" (at 101.2 115.4) (layer "F.SilkS")
     (effects (font (size 1 1) (thickness 0.125)) (justify left))
